File: Electronics/vvfd.kicad_sch (KiCad schematic)
At the start: 58 parts, among them J1 USB_C_Receptacle_USB2.0_14P, J2 Conn_01x02_Pin, J3 Conn_02x05_Counter_Clockwise, J4 Conn_02x05_Counter_Clockwise, J5 Conn_02x05_Counter_Clockwise, Q1 IRLU014PBF, Q2 IRLU014PBF, Q3 IRLU014PBF, Q4 IRLU014PBF, Q5 IRLU014PBF, Q6 IRLU014PBF, U1 MC34063AD, U2 TLV274

Commit message: Fixed ERC and DRC
Changed lines of the file:
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@@
 	(text "High Current Sense"
 		(exclude_from_sim no)
-		(at 271.78 334.518 0)
+		(at 271.78 336.55 0)
 		(effects
 			(font
@@
 	(text "Low Current Sense"
 		(exclude_from_sim no)
-		(at 271.78 267.208 0)
+		(at 272.034 269.494 0)
 		(effects
 			(font
@@
 		)
 	)
-	(label "LCS"
-		(at 269.24 270.51 0)
-		(effects
-			(font
-				(size 1.27 1.27)
-			)
-			(justify left bottom)
-		)
-	)
 	(label "LCS_DRAIN"
 		(at 251.46 284.48 0)
@@
 		)
 	)
-	(label "HCS"
-		(at 269.24 337.82 0)
-		(effects
-			(font
-				(size 1.27 1.27)
-			)
-			(justify left bottom)
-		)
-	)
 	(label "HCS_GATE"
 		(at 233.68 358.14 0)
@@
 		)
 		(instances
-			(project "vfd"
+			(project "vvfd"
 				(path "/36e0811c-69c7-4576-98bb-165d7651c83d"
 					(reference "#FLG02")

Commit message: Added filament timer
Added a timer to control the filament h-brdige on the main PCB.
Also added some more decoupling capacitors, but some have dubious
placement. Still better than nothing.
Parts:
- added C1, C11: 100n, Capacitor_THT:C_Disc_D5.1mm_W3.2mm_P5.00mm, symbol Device:C
- added C10, C5: 220n, Capacitor_THT:C_Disc_D5.1mm_W3.2mm_P5.00mm, symbol Device:C
- added C4: 1n, Capacitor_THT:C_Disc_D5.1mm_W3.2mm_P5.00mm, symbol Device:C
- added C6, C7: 10n, Capacitor_THT:C_Disc_D5.1mm_W3.2mm_P5.00mm, symbol Device:C
- added R10: 68k, Resistor_THT:R_Axial_DIN0207_L6.3mm_D2.5mm_P2.54mm_Vertical, symbol Device:R
- added R2: 33k, Resistor_THT:R_Axial_DIN0207_L6.3mm_D2.5mm_P2.54mm_Vertical, symbol Device:R
- added R5: 39k, Resistor_THT:R_Axial_DIN0207_L6.3mm_D2.5mm_P2.54mm_Vertical, symbol Device:R
- added R8: 1k, Resistor_THT:R_Axial_DIN0207_L6.3mm_D2.5mm_P2.54mm_Vertical, symbol Device:R
- added U1: LM556, Package_DIP:DIP-14_W7.62mm, symbol Timer:LM556
- renumbered C5 to C12, C1 to C2, C2 to C3, C3 to C8, C4 to C9, J5 to J4, J4 to J5, R7 to R11, R8 to R12, R9 to R13, R10 to R14, R11 to R15, R12 to R16, R13 to R17, R14 to R18, R15 to R19, R16 to R20, R17 to R21, R18 to R22, R19 to R23, R20 to R24, R21 to R25, R22 to R26, R23 to R27, R24 to R28, R25 to R29, R2 to R3, R3 to R4, R4 to R6, R5 to R7, R6 to R9, TP3 to TP1, TP4 to TP2, TP2 to TP3, TP1 to TP4, U1 to U2, U2 to U3
Connections:
- net +5V: now also J4.8 (Pin_8)
- net GND: now also J4.4 (Pin_4), C1.2, C10.2, C11.2, C5.2, C6.2, C7.2, U1.7 (GND), U1.7 (GND)
- net H1: now also C4.1, U1.5 (Q); no longer J4.8 (Pin_8)
- net H2: now also U1.9 (Q); no longer J4.4 (Pin_4)
- net VCC: now also C1.1, C11.1, R2.1, R5.1, R8.1, U1.10 (R), U1.14 (VCC), U1.14 (VCC), U1.4 (R)
- new net TIMING_CAP_1: C10.1, R10.2, U1.2 (THR), U1.6 (TR)
- new net TIMING_CAP_2: C5.1, R5.2, U1.12 (THR), U1.13 (DIS)
- new net TIM_1_CV: C6.1, U1.3 (CV)
- new net TIM_1_DIS: R10.1, R8.2, U1.1 (DIS)
- new net TIM_2_CV: C7.1, U1.11 (CV)
- new net TIM_2_IN: C4.2, R2.2, U1.8 (TR)
Other:
- note added: "Creates a clock for H1 and H2"
- note added: "H-bridge timer"
- note added: "H1 and H2 are used to turn on different H-bridge polarities They should never be on at the same time, otherwise they will create a short circuit"
- note added: "IRLU014PBF Digi with better specs RFD14N05L UC one"
- note added: "t_h = 0.693 * (68k + 1k) * 220n = 10.5ms t_l = 0.693 * 68k * 220n = 10.4ms"
- note added: "t_p = 1.1 * 39k * 220n = 9.4ms"
- note removed: "IRLU014PBF Digi with better specs"
- note removed: "It's up to the MCU to control H1 and H2 They should NOT be on at the same time"
- note removed: "RFD14N05L UC one"
- moved on the sheet: C12, C2, C3, C8, C9, D1, D2, F1, F2, H1, H2, H3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

Commit message: Added VFD output pulldowns
Added pulldowns and more decoupling capacitors. The capacitors and
pulldowns can probably be omitted, but I've put them in for more flexibility.
Parts:
- C10, C4, C5, C6, C7: Cascade Component (none) -> 0; Digikey Part No (none) -> UC; Master Component (none) -> 1; Unit Price ($) (none) -> 0.20
- R10, R2, R5, R8: Cascade Component (none) -> 0; Digikey Part No (none) -> UC; Master Component (none) -> 1; Unit Price ($) (none) -> 0.00
- U1: Cascade Component (none) -> 0; Digikey Part No (none) -> UC; Manufacturer Part No (none) -> LM557; Master Component (none) -> 1; Unit Price ($) (none) -> 1.00

Commit message: Fixed H-bridge
Old H-bridge was the wrong type, changed to using some P-channel
mosfets. Also fixed the cost spreadsheet.
Parts:
- removed F2: 500mA hold, Fuse:Fuse_Littelfuse_395Series, symbol Device:Polyfuse
- removed Q1, Q2, Q3, Q4, Q5, Q6: IRLU014PBF, Package_TO_SOT_THT:TO-251-3_Vertical, symbol Transistor_FET:IRF540N
- added Q1, Q2: DMG2305UX, Package_TO_SOT_SMD:SOT-23, symbol Transistor_FET:DMG2301L
- added Q3, Q4, Q5, Q6: SL3402, Package_TO_SOT_SMD:SOT-23, symbol Transistor_FET:DMN24H3D5L
- R11, R12, R13, R14: footprint Resistor_THT:R_Axial_DIN0207_L6.3mm_D2.5mm_P2.54mm_Vertical -> Resistor_THT:R_Axial_DIN0207_L6.3mm_D2.5mm_P7.62mm_Horizontal
- R23: Cascade Component 1 -> 0; Master Component 0 -> 1
Connections:
- net +5V: now also Q1.2 (S), Q2.2 (S)
- net BRIDGE_G1: now also Q2.1 (G), Q4.1 (G)
- net BRIDGE_G2: now also Q1.1 (G), Q3.1 (G)
- net FILAMENT_1: now also Q1.3 (D), Q3.3 (D)
- net FILAMENT_2: now also Q2.3 (D), Q4.3 (D)
- net GND: now also Q3.2 (S), Q4.2 (S), Q5.2 (S), Q6.2 (S)
- net HCS_DRAIN: now also Q6.3 (D)
- net HCS_GATE: now also Q6.1 (G)
- net LCS_DRAIN: now also Q5.3 (D)
- net LCS_GATE: now also Q5.1 (G)
Other:
- note added: "H1 and H2 are used to turn on different H-bridge polarities"
- note removed: "H1 and H2 are used to turn on different H-bridge polarities They should never be on at the same time, otherwise they will create a short circuit"
- note removed: "IRLU014PBF Digi with better specs RFD14N05L UC one"
- moved on the sheet: J2, R11, R12, R13, R14

Commit message: Added timer circuit test picture
Added a picture of the timer circuits output recorded on an oscilloscope
Parts:
- C10, C5: Unit Price ($) 0.20 -> 0.40
