File: DriverBoard/vfd_drive.kicad_sch (KiCad schematic)
At the start: 6 parts, among them J6 Conn_01x08_Pin, U4 74HC595, U5 TBD62783A

Commit message: Removed Current Sensing
Removed current sensing, because it would require a major design
overhaul to work properly.
Parts:
- renumbered C13 to C16, C14 to C17, J6 to J5
Connections:
- net GNDA is gone; now on net GND: C17.2, RN1.1 (common), U5.10 (GND)
