File: Shield/VVFDShield.kicad_pcb (KiCad board)
At the start: 2 copper layers, 68.6 x 53.3 mm, 18 parts, among them J1 Conn_02x05_Counter_Clockwise, J2 Conn_02x05_Counter_Clockwise, P1 Power, P2 Digital, P3 Digital, P4 Analog, SW1 SW_SPST, SW2 SW_SPST

Commit message: Removed Current Sensing
Removed current sensing, because it would require a major design
overhaul to work properly.
Parts:
- removed J2: Conn_02x05_Counter_Clockwise, Connector_IDC:IDC-Header_2x05_P2.54mm_Vertical
- moved R2 5.68 mm to (159.2, 103.0)
- moved R4 5.68 mm to (159.2, 106.2)
- renumbered J1 to J5
Connections:
- J5 pad 10: unconnected-(J1-Pin_10-Pad10) -> +5V
- J5 pad 5: +5V -> unconnected-(J5-Pin_5-Pad5)
- J5 pad 9: unconnected-(J1-Pin_9-Pad9) -> +5V
- P3 pad 3: LCS_EN -> /D5
- P3 pad 4: HCS_EN -> /D4
- P4 pad 1: 3HCS -> /A0
- P4 pad 2: 5HCS -> /A1
- P4 pad 3: 3LCS -> /A2
- P4 pad 4: 5LCS -> /A3
Routing:
- net LCS_EN: track 38.1 -> 0.00 mm
- net HCS_EN: track 37.2 -> 0.00 mm
- net 5LCS: track 30.9 -> 0.00 mm, vias 2 -> 0
- net 3LCS: track 30.3 -> 0.00 mm, vias 2 -> 0
- net 5HCS: track 16.6 -> 0.00 mm
- net 3HCS: track 13.7 -> 0.00 mm
- net BUTTON_2: track 27.0 -> 31.8 mm
- net /TAC2: track 36.3 -> 31.6 mm
- net /TAC1: track 38.5 -> 33.7 mm
- net BUTTON_1: track 23.5 -> 27.5 mm
- net +5V: track 92.4 -> 89.9 mm
Other:
- board text removed: "(Hide User.ArduinoUnoR3 Layer to make invisible)"
- board text removed: "Arduino Uno R3 Keepouts"
- board text removed: "CASCADE IN"
- board text removed: "MCU ONLY I/O"
- board text removed: "Shield Template 2025-01-15"
